File: MicroMod_Extension.sch (KiCad schematic (older format))
At the start: 81 parts, among them J1 2199230-4, J10 2199230-4, J2 XKB_U262-16XN-4BVC11, J3 RSP-122811-01, J4 Screw_Terminal_01x04, J5 Conn_01x08, J6 Conn_01x08, J7 Conn_01x02, J8 Conn_01x04, J9 Conn_01x04, SW1 TL1014BF160QG, U1 24aa64ft-eot, U2 nRF51822-QFAA-R7, U3 RFX2411N, U4 TPS62170DSG, U5 NCP702SN30T1G, U6 NCP702SN30T1G, U7 BMI270, U8 BMP384, Y1 TSX-3225_16.0000MF18X-AC3

Commit message: update pcb
Parts:
- removed C10: 1u, Capacitor_SMD:C_0402_1005Metric, symbol Device:C
- removed C8: 100n, Capacitor_SMD:C_0402_1005Metric, symbol Device:C
- removed J10: 2199230-4, MicroMod_Extension:M.2-CARD-E-22, symbol MicroMod_Extension:2199230-4
- J4: footprint Connector_PinHeader_2.54mm:PinHeader_1x04_P2.54mm_Vertical -> Connector_JST:JST_SUR_SM04B-SURS-TF_1x04-1MP_P0.80mm_Horizontal
- J5, J6: footprint MicroMod_Extension:JST_SUR_BM08B-SURS-TF_1x08-1MP_P0.80mm_Vertical -> Connector_JST:JST_SUR_BM08B-SURS-TF_1x08-1MP_P0.80mm_Vertical
- J8, J9: footprint MicroMod_Extension:JST_SUR_BM04B-SURS-TF_1x04-1MP_P0.80mm_Vertical -> Connector_JST:JST_SUR_SM04B-SURS-TF_1x04-1MP_P0.80mm_Horizontal
- TP4, TP5, TP6, TP7: value TestPoint -> Mount Hole
- TP8: value TestPoint -> Mount Hole; footprint MicroMod_Extension:97730256330R -> Mounting_Wuerth:Mounting_Wuerth_WA-SMSI-M2_H2.5mm_9774025243
Connections:
- net VCC: no longer J8.1 (Pin_1), J9.1 (Pin_1)
- no-connect marks 39 -> 41
Changed lines of the file:
@@
-$EndComp
-$Comp
-L Device:C C8
-U 1 1 6180E744
-P 14900 8375
-F 0 "C8" H 15015 8421 50  0000 L CNN
-F 1 "100n" H 15015 8330 50  0000 L CNN
-F 2 "Capacitor_SMD:C_0402_1005Metric" H 14938 8225 50  0001 C CNN
-F 3 "~" H 14900 8375 50  0001 C CNN
-	1    14900 8375
-	1    0    0    -1
 $EndComp
 $Comp
@@
 	14575 8100 14900 8100
 Wire Wire Line
-	14900 8100 14900 8225
-Wire Wire Line
 	15200 8100 15200 8225
 Connection ~ 14900 8100
@@
 Wire Wire Line
 	14575 8625 14900 8625
-Wire Wire Line
-	14900 8625 14900 8525
 Wire Wire Line
 	14900 8625 15200 8625
@@
 	14275 8625 14575 8625
 Connection ~ 14575 8625
-$Comp
-L Device:C C10
-U 1 1 621F1946
-P 15525 8375
-F 0 "C10" H 15640 8421 50  0000 L CNN
-F 1 "1u" H 15640 8330 50  0000 L CNN
-F 2 "Capacitor_SMD:C_0402_1005Metric" H 15563 8225 50  0001 C CNN
-F 3 "~" H 15525 8375 50  0001 C CNN
-	1    15525 8375
-	1    0    0    -1
-$EndComp
-Wire Wire Line
-	15525 8225 15525 8100
 Wire Wire Line
 	14900 8100 15200 8100
-Connection ~ 15200 8100
-Wire Wire Line
-	15200 8100 15525 8100
-Wire Wire Line
-	15525 8625 15525 8525
-Wire Wire Line
-	15200 8625 15525 8625
-Connection ~ 15200 8625
 Wire Wire Line
 	11150 5225 11150 5325
@@
 F 0 "J4" H 15505 5267 50  0000 L CNN
 F 1 "Screw_Terminal_01x04" H 15505 5176 50  0000 L CNN
-F 2 "Connector_PinHeader_2.54mm:PinHeader_1x04_P2.54mm_Vertical" H 15425 5275 50  0001 C CNN
+F 2 "Connector_JST:JST_SUR_SM04B-SURS-TF_1x04-1MP_P0.80mm_Horizontal" H 15425 5275 50  0001 C CNN
 F 3 "~" H 15425 5275 50  0001 C CNN
 	1    15425 5275
@@
 F 0 "J5" H 15505 1967 50  0000 L CNN
 F 1 "Conn_01x08" H 15505 1876 50  0000 L CNN
-F 2 "MicroMod_Extension:JST_SUR_BM08B-SURS-TF_1x08-1MP_P0.80mm_Vertical" H 15425 1975 50  0001 C CNN
+F 2 "Connector_JST:JST_SUR_BM08B-SURS-TF_1x08-1MP_P0.80mm_Vertical" H 15425 1975 50  0001 C CNN
 F 3 "~" H 15425 1975 50  0001 C CNN
 	1    15425 1975
@@
 F 0 "J6" H 15505 3017 50  0000 L CNN
 F 1 "Conn_01x08" H 15505 2926 50  0000 L CNN
-F 2 "MicroMod_Extension:JST_SUR_BM08B-SURS-TF_1x08-1MP_P0.80mm_Vertical" H 15425 3025 50  0001 C CNN
+F 2 "Connector_JST:JST_SUR_BM08B-SURS-TF_1x08-1MP_P0.80mm_Vertical" H 15425 3025 50  0001 C CNN
 F 3 "~" H 15425 3025 50  0001 C CNN
 	1    15425 3025
@@
 F 0 "J8" H 15505 3967 50  0000 L CNN
 F 1 "Conn_01x04" H 15505 3876 50  0000 L CNN
-F 2 "MicroMod_Extension:JST_SUR_BM04B-SURS-TF_1x04-1MP_P0.80mm_Vertical" H 15425 3975 50  0001 C CNN
+F 2 "Connector_JST:JST_SUR_SM04B-SURS-TF_1x04-1MP_P0.80mm_Horizontal" H 15425 3975 50  0001 C CNN
 F 3 "~" H 15425 3975 50  0001 C CNN
 	1    15425 3975
@@
 	0    1    1    0
 $EndComp
-Text Label 15225 3875 2    50   ~ 0
-VCC
 Text Label 15225 3975 2    50   ~ 0
 E_RX1
@@
 F 0 "J9" H 15505 4617 50  0000 L CNN
 F 1 "Conn_01x04" H 15505 4526 50  0000 L CNN
-F 2 "MicroMod_Extension:JST_SUR_BM04B-SURS-TF_1x04-1MP_P0.80mm_Vertical" H 15425 4625 50  0001 C CNN
+F 2 "Connector_JST:JST_SUR_SM04B-SURS-TF_1x04-1MP_P0.80mm_Horizontal" H 15425 4625 50  0001 C CNN
 F 3 "~" H 15425 4625 50  0001 C CNN
 	1    15425 4625
@@
 	0    1    1    0
 $EndComp
-Text Label 15225 4525 2    50   ~ 0
-VCC
 Text Label 15225 4625 2    50   ~ 0
 E_RX2
@@
 P 14925 1200
 F 0 "TP4" H 14983 1318 50  0000 L CNN
-F 1 "TestPoint" H 14983 1227 50  0000 L CNN
+F 1 "Mount Hole" H 14900 1050 50  0000 L CNN
 F 2 "TestPoint:TestPoint_Plated_Hole_D3.0mm" H 15125 1200 50  0001 C CNN
 F 3 "~" H 15125 1200 50  0001 C CNN
@@
 P 15150 1200
 F 0 "TP5" H 15208 1318 50  0000 L CNN
-F 1 "TestPoint" H 15208 1227 50  0000 L CNN
+F 1 "Mount Hole" H 15125 1000 50  0000 L CNN
 F 2 "TestPoint:TestPoint_Plated_Hole_D3.0mm" H 15350 1200 50  0001 C CNN
 F 3 "~" H 15350 1200 50  0001 C CNN
@@
 P 15350 1200
 F 0 "TP6" H 15408 1318 50  0000 L CNN
-F 1 "TestPoint" H 15408 1227 50  0000 L CNN
+F 1 "Mount Hole" H 15325 1125 50  0000 L CNN
 F 2 "TestPoint:TestPoint_Plated_Hole_D3.0mm" H 15550 1200 50  0001 C CNN
 F 3 "~" H 15550 1200 50  0001 C CNN
@@
 P 15575 1200
 F 0 "TP7" H 15633 1318 50  0000 L CNN
-F 1 "TestPoint" H 15633 1227 50  0000 L CNN
+F 1 "Mount Hole" H 15550 1050 50  0000 L CNN
 F 2 "TestPoint:TestPoint_Plated_Hole_D3.0mm" H 15775 1200 50  0001 C CNN
 F 3 "~" H 15775 1200 50  0001 C CNN
@@
 $EndComp
 $Comp
-L MicroMod_Extension:2199230-4 J10
-U 1 1 61980F5E
-P 13625 3700
-F 0 "J10" H 13625 5767 50  0000 C CNN
-F 1 "2199230-4" H 13625 5676 50  0000 C CNN
-F 2 "MicroMod_Extension:M.2-CARD-E-22" H 13625 3700 50  0001 L BNN
-F 3 "" H 13625 3700 50  0001 L BNN
-F 4 "Compliant" H 13625 3700 50  0001 L BNN "EU_RoHS_Compliance"
-F 5 "2199230-4" H 13625 3700 50  0001 L BNN "Comment"
-	1    13625 3700
-	1    0    0    -1
-$EndComp
-$Comp
 L Connector:TestPoint TP8
 U 1 1 6199C5E3
 P 14775 1200
 F 0 "TP8" H 14833 1318 50  0000 L CNN
-F 1 "TestPoint" H 14833 1227 50  0000 L CNN
-F 2 "MicroMod_Extension:97730256330R" H 14975 1200 50  0001 C CNN
+F 1 "Mount Hole" H 14750 1125 50  0000 L CNN
+F 2 "Mounting_Wuerth:Mounting_Wuerth_WA-SMSI-M2_H2.5mm_9774025243" H 14975 1200 50  0001 C CNN
 F 3 "~" H 14975 1200 50  0001 C CNN
 	1    14775 1200
@@
 	14775 1200 14925 1200
 Connection ~ 14925 1200
+NoConn ~ 15225 3875
+NoConn ~ 15225 4525
 $EndSCHEMATC
