File: MicroMod_Extension.kicad_pcb (KiCad board)
At the start: 2 copper layers, 1 part, among them J1 2199230-4

Commit message: inductor type
Parts:
- added C1: 100n, Capacitor_SMD:C_0402_1005Metric, F.Cu at (133.8, 81.8)
- added C2: 100n, Capacitor_SMD:C_0402_1005Metric, F.Cu at (153.8, 71.8)
- added C3: 100n, Capacitor_SMD:C_0402_1005Metric, F.Cu at (136.7, 81.8)
- added C4: 47n, Capacitor_SMD:C_0402_1005Metric, F.Cu at (139.6, 81.8)
- added C5: 100n, Capacitor_SMD:C_0402_1005Metric, F.Cu at (142.5, 81.8)
- added J2: XKB_U262-16XN-4BVC11, Connector_USB:USB_C_Receptacle_XKB_U262-16XN-4BVC11, F.Cu at (134.3, 73.3)
- added U1: 24aa64ft-eot, Package_TO_SOT_SMD:SOT-23-5, F.Cu at (152.2, 81.4)
- added U2: nRF51822-QFAA-R7, Package_DFN_QFN:QFN-48-1EP_6x6mm_P0.4mm_EP4.6x4.6mm, F.Cu at (148.2, 74.9)
- added Y1: TSX-3225_16.0000MF18X-AC3, MicroMod_Extension:XTAL_TSX-3225_16.0000MF18X-AC3, F.Cu at (147.2, 81.2)
Connections:
- net Net-(J1-Pad10) renamed /C8
- net Net-(J1-Pad11) renamed /IMU_SDA
- net Net-(J1-Pad12) renamed /B12
- net Net-(J1-Pad13) renamed /IMU_SCL
- net Net-(J1-Pad14) renamed /MOTOR1
- net Net-(J1-Pad15) renamed /SPI2_CLK
- net Net-(J1-Pad16) renamed /NRF_CTRL
- net Net-(J1-Pad17) renamed /SPI2_MISO
- net Net-(J1-Pad19) renamed /SPI2_MOSI
- net Net-(J1-Pad20) renamed /GREEN_R
- net Net-(J1-Pad21) renamed /MOTOR2
- net Net-(J1-Pad22) renamed /RED_R
- net Net-(J1-Pad23) renamed /B10
- net Net-(J1-Pad32) renamed /B4
- net Net-(J1-Pad34) renamed /E_SPI_MOSI
- net Net-(J1-Pad35) renamed /INT_GYR
- net Net-(J1-Pad36) renamed /E_SPI_MISO
- net Net-(J1-Pad37) renamed /B1
- net Net-(J1-Pad38) renamed /E_SPI_CLK
- net Net-(J1-Pad39) renamed /B0
- net Net-(J1-Pad41) renamed /C5
- net Net-(J1-Pad43) renamed /C4
- net Net-(J1-Pad44) renamed /E_TX1
- net Net-(J1-Pad45) renamed /A0
- net Net-(J1-Pad46) renamed /E_RX1
- net Net-(J1-Pad47) renamed /C13
- net Net-(J1-Pad48) renamed /E_RX2
- net Net-(J1-Pad49) renamed /B5
- net Net-(J1-Pad50) renamed /E_TX2
- net Net-(J1-Pad51) renamed /B8
- net Net-(J1-Pad52) renamed /C12
- net Net-(J1-Pad54) renamed /C15
- net Net-(J1-Pad6) renamed /NRF_TX
- net Net-(J1-Pad61) renamed /STM_SWCLK
- net Net-(J1-Pad65) renamed /STM_SWIO
- net Net-(J1-Pad66) renamed /GREEN_L
- net Net-(J1-Pad67) renamed /NRST
- net Net-(J1-Pad68) renamed /RED_L
- net Net-(J1-Pad69) renamed /STM_SWO
- net Net-(J1-Pad7) renamed /OTG_FS_ID
- net Net-(J1-Pad70) renamed /BOOT0
- net Net-(J1-Pad71) renamed /MOTOR3
- net Net-(J1-Pad72) renamed /MOTOR4
- net Net-(J1-Pad8) renamed /NRF_RX
- net Net-(J1-Pad9) renamed /OTG_FS_VBUS
- J1 pad 1: Net-(J1-Pad1) -> /VCC
- J1 pad 18: Net-(J1-Pad18) -> GND
- J1 pad 2: Net-(J1-Pad2) -> /VCC
- J1 pad 3: Net-(J1-Pad3) -> /OTG_FS_D+
- J1 pad 33: Net-(J1-Pad33) -> GND
- J1 pad 4: Net-(J1-Pad4) -> GND
- J1 pad 40: Net-(J1-Pad40) -> /E_SCL
- J1 pad 42: Net-(J1-Pad42) -> /E_SDA
- J1 pad 5: Net-(J1-Pad5) -> /OTG_FS_D-
- J1 pad 59: Net-(J1-Pad59) -> /VCC
- J1 pad 63: Net-(J1-Pad63) -> GND
- J1 pad 73: Net-(J1-Pad73) -> /VBAT
- J1 pad 74: Net-(J1-Pad74) -> GND
- J1 pad 75: Net-(J1-Pad75) -> /VCC
- J1 pad S1: Net-(J1-PadS1) -> GND
- J1 pad S2: Net-(J1-PadS1) -> GND

Commit message: update RF
Parts:
- added C6: 220p, Capacitor_SMD:C_0402_1005Metric, F.Cu at (123.2, 83.6)
- added C7: 1u, Capacitor_SMD:C_0402_1005Metric, F.Cu at (122.6, 86.7)
- added FL1: 2450BM14E0003T, MicroMod_Extension:FIL_2450BM14E0003T, F.Cu at (120.3, 84.2)
- added L1: 2nH, Inductor_SMD:L_0402_1005Metric, F.Cu at (119.7, 86.7)
- added U3: RFX2411N, Package_DFN_QFN:QFN-20-1EP_3x3mm_P0.45mm_EP1.6x1.6mm, F.Cu at (158.8, 89.9)
Other:
- net class Default: clearance 0.2 -> 0.2032; trace_width 0.25 -> 0.127; via_dia 0.8 -> 0.6096; via_drill 0.4 -> 0.3048
- rule trace_clearance: 0.2 -> 0.2032
- rule trace_min: 0.2 -> 0.127
- rule via_min_drill: 0.3 -> 0.254
- rule via_min_size: 0.4 -> 0.381

Commit message: add power management
Parts:
- added C10: 1u, Capacitor_SMD:C_0402_1005Metric, F.Cu at (192.5, 79.4)
- added C11: 2.5p, Capacitor_SMD:C_0402_1005Metric, F.Cu at (190.6, 85.4)
- added C12: 10u, Capacitor_SMD:C_0402_1005Metric, F.Cu at (187.7, 87.4)
- added C13: 10n, Capacitor_SMD:C_0402_1005Metric, F.Cu at (184.8, 89.4)
- added C14: 220p, Capacitor_SMD:C_0402_1005Metric, F.Cu at (191.5, 83.5)
- added C15: 4.7u, Capacitor_SMD:C_0402_1005Metric, F.Cu at (181.9, 91.9)
- added C16: 220p, Capacitor_SMD:C_0402_1005Metric, F.Cu at (187.7, 85.5)
- added C17: 2.2n, Capacitor_SMD:C_0402_1005Metric, F.Cu at (184.9, 87.4)
- added C18: 22u, Capacitor_SMD:C_0402_1005Metric, F.Cu at (191.7, 81.4)
- added C19: 1u, Capacitor_SMD:C_0402_1005Metric, F.Cu at (181.9, 90.0)
- added C20: 1u, Capacitor_SMD:C_0402_1005Metric, F.Cu at (181.9, 88.0)
- added C21: 1u, Capacitor_SMD:C_0402_1005Metric, F.Cu at (188.8, 81.5)
- added C22: 1u, Capacitor_SMD:C_0402_1005Metric, F.Cu at (188.6, 83.5)
- added C8: 100n, Capacitor_SMD:C_0402_1005Metric, F.Cu at (192.5, 77.4)
- added C9: 10n, Capacitor_SMD:C_0402_1005Metric, F.Cu at (184.9, 85.5)
- added D1: LED, MicroMod_Extension:LED-0603, F.Cu at (162.5, 92.4)
- added D2: 150066RG74000, MicroMod_Extension:150066RG74000, F.Cu at (179.1, 79.6)
- added D3: SMF4L17A, Diode_SMD:D_SOD-123, F.Cu at (163.5, 85.2)
- added D4: 150066RG74000, MicroMod_Extension:150066RG74000, F.Cu at (174.1, 83.4)
- added D5: MBR0520-TP, Diode_SMD:D_SOD-123, F.Cu at (172.3, 76.1)
- added E1: 2450AT18B100E, MicroMod_Extension:XDCR_2450AT18B100E, F.Cu at (164.1, 82.0)
- added FL2: ADFC15-2450.00-A-T, MicroMod_Extension:FIL_ADFC15-2450.00-A-T, F.Cu at (186.5, 75.9)
- added FL3: ADFC15-2450.00-A-T, MicroMod_Extension:FIL_ADFC15-2450.00-A-T, F.Cu at (178.1, 84.1)
- added J3: RSP-122811-01, MicroMod_Extension:SAMTEC_RSP-122811-01, F.Cu at (169.8, 82.5)
- added L2: 2nH, Inductor_SMD:L_0402_1005Metric, F.Cu at (182.0, 86.0)
- added L3: 1nH, Inductor_SMD:L_0402_1005Metric, F.Cu at (170.9, 78.8)
- added L4: 2nH, Inductor_SMD:L_0402_1005Metric, F.Cu at (189.6, 75.4)
- added L5: 2.2uH-TYA2520102R2M-10, Inductor_SMD:L_1008_2520Metric, F.Cu at (175.0, 80.8)
- added R1: 150r, Resistor_SMD:R_0402_1005Metric, F.Cu at (182.8, 82.0)
- added R10: 150r, Resistor_SMD:R_0402_1005Metric, F.Cu at (189.3, 79.4)
- added R11: 510k, Resistor_SMD:R_0402_1005Metric, F.Cu at (170.4, 92.1)
- added R12: 110k, Resistor_SMD:R_0402_1005Metric, F.Cu at (176.2, 90.6)
- added R13: 10K, Resistor_SMD:R_0402_1005Metric, F.Cu at (185.8, 83.5)
- added R14: 430K, Resistor_SMD:R_0402_1005Metric, F.Cu at (176.2, 87.2)
- added R15: 82K, Resistor_SMD:R_0402_1005Metric, F.Cu at (192.5, 75.4)
- added R2: 5.1k, Resistor_SMD:R_0402_1005Metric, F.Cu at (185.9, 81.5)
- added R3: 5.1k, Resistor_SMD:R_0402_1005Metric, F.Cu at (181.3, 84.0)
- added R4: 10K, Resistor_SMD:R_0402_1005Metric, F.Cu at (189.6, 77.4)
- added R5: 150r, Resistor_SMD:R_0402_1005Metric, F.Cu at (173.3, 90.3)
- added R6: 10K, Resistor_SMD:R_0402_1005Metric, F.Cu at (179.1, 86.6)
- added R7: 10K, Resistor_SMD:R_0402_1005Metric, F.Cu at (173.3, 92.3)
- added R8: 150r, Resistor_SMD:R_0402_1005Metric, F.Cu at (179.1, 88.6)
- added R9: 150r, Resistor_SMD:R_0402_1005Metric, F.Cu at (176.2, 92.6)
- added SW1: TL1014BF160QG, MicroMod_Extension:E-Switch-TL1014BF160QG-0, F.Cu at (164.6, 76.9)
- added TP1: TestPoint, TestPoint:TestPoint_Pad_D1.0mm, F.Cu at (186.3, 79.0)
- added TP2: TestPoint, TestPoint:TestPoint_Pad_D1.0mm, F.Cu at (182.9, 79.5)
- added TP3: TestPoint, TestPoint:TestPoint_Pad_D1.0mm, F.Cu at (173.2, 87.8)
- added U4: TPS62170DSG, Package_SON:WSON-8-1EP_2x2mm_P0.5mm_EP0.9x1.6mm_ThermalVias, F.Cu at (182.7, 76.2)
- added U5: NCP702SN30T1G, Package_TO_SOT_SMD:TSOT-23-5, F.Cu at (177.8, 76.7)
- added U6: NCP702SN30T1G, Package_TO_SOT_SMD:TSOT-23-5, F.Cu at (163.3, 89.1)
- C2, C3: value 100n -> 12p
- C6: value 220p -> 100n
- C7: value 1u -> 100n
- L1: value 2nH -> 4.7nH
- U3: footprint Package_DFN_QFN:QFN-20-1EP_3x3mm_P0.45mm_EP1.6x1.6mm -> Package_DFN_QFN:QFN-20-1EP_3x3mm_P0.4mm_EP1.65x1.65mm
- moved C7 56.6 mm to (179.1, 90.6)
- moved C6 56.6 mm to (179.1, 92.6)
- moved L1 48.1 mm to (167.4, 92.1)
- moved U3 10.4 mm to (169.0, 88.4)
Connections:
- net /E_SPI_CLK renamed /E_SPI_SCK
- net /SPI2_CLK renamed /SPI2_SCK
- C6 pad 1: Net-(C6-Pad1) -> /VCC_NRF
- C7 pad 1: Net-(C6-Pad1) -> /VCC_NRF
- J1 pad 67: /NRST -> /STM_NRST
- J1 pad 70: /BOOT0 -> /STM_BOOT0
- J1 pad 73: /VBAT -> /VCC_NRF
- J1 pad 9: /OTG_FS_VBUS -> VBUS
- J2 pad A4: /VBUS -> VBUS
- J2 pad A9: /VBUS -> VBUS
- J2 pad B4: /VBUS -> VBUS
- J2 pad B9: /VBUS -> VBUS
- L1 pad 1: GND -> Net-(E1-Pad1)
- L1 pad 2: Net-(L1-Pad2) -> Net-(C11-Pad1)
- U2 pad 1: /VBAT -> /VCC_NRF
- U2 pad 12: /VBAT -> /VCC_NRF
- U2 pad 16: Net-(U2-Pad16) -> /VEN_D
- U2 pad 19: Net-(U2-Pad19) -> /LED_BLUE
- U2 pad 20: Net-(U2-Pad20) -> /NRF_CTRL
- U2 pad 25: Net-(U2-Pad25) -> /SWITCH
- U2 pad 26: Net-(U2-Pad26) -> /PA_SW_ANT
- U2 pad 27: Net-(U2-Pad27) -> /PA_MODE
- U2 pad 28: Net-(U2-Pad28) -> /PA_RXEN
- U2 pad 3: Net-(U2-Pad3) -> /NRF_RX
- U2 pad 35: /VBAT -> /VCC_NRF
- U2 pad 36: /VBAT -> /VCC_NRF
- U2 pad 40: Net-(U2-Pad40) -> /STM_NRST
- U2 pad 41: Net-(U2-Pad41) -> /STM_BOOT0
- U2 pad 48: Net-(U2-Pad48) -> /NRF_TX
- U2 pad 5: Net-(U2-Pad5) -> /VBAT
- U2 pad 8: Net-(U2-Pad8) -> /PM_PGOOD
- U3 pad 10: Net-(U3-Pad10) -> /PA_SW_ANT
- U3 pad 15: Net-(L1-Pad2) -> Net-(L4-Pad1)
- U3 pad 18: Net-(C6-Pad1) -> /VCC_NRF
- U3 pad 2: Net-(U3-Pad2) -> GND
- U3 pad 20: Net-(C6-Pad1) -> /VCC_NRF
- U3 pad 4: Net-(U3-Pad4) -> GND
- U3 pad 5: Net-(U3-Pad5) -> Net-(FL1-Pad1)
- U3 pad 7: Net-(U3-Pad7) -> /PA_RXEN
- U3 pad 9: Net-(U3-Pad9) -> /PA_MODE

Commit message: update pcb
Parts:
- removed R4: 10K, Resistor_SMD:R_0402_1005Metric
- added C23: 100n, Capacitor_SMD:C_0402_1005Metric, F.Cu at (155.5, 109.9)
- added C24: 100n, Capacitor_SMD:C_0402_1005Metric, F.Cu at (158.0, 109.9)
- added C25: 4.7u, Capacitor_SMD:C_0402_1005Metric, F.Cu at (205.6, 114.9)
- added J4: Screw_Terminal_01x04, Connector_PinHeader_2.54mm:PinHeader_1x04_P2.54mm_Vertical, F.Cu at (154.8, 130.3)
- added J5: Conn_01x08, MicroMod_Extension:JST_SUR_BM08B-SURS-TF_1x08-1MP_P0.80mm_Vertical, F.Cu at (158.0, 86.1)
- added J6: Conn_01x08, MicroMod_Extension:JST_SUR_BM08B-SURS-TF_1x08-1MP_P0.80mm_Vertical, F.Cu at (158.0, 91.0)
- added J7: Conn_01x02, Connector_PinHeader_2.54mm:PinHeader_1x02_P2.54mm_Vertical, F.Cu at (166.0, 86.0)
- added J8: Conn_01x04, MicroMod_Extension:JST_SUR_BM04B-SURS-TF_1x04-1MP_P0.80mm_Vertical, F.Cu at (138.9, 82.4)
- added J9: Conn_01x04, MicroMod_Extension:JST_SUR_BM04B-SURS-TF_1x04-1MP_P0.80mm_Vertical, F.Cu at (138.9, 87.3)
- added U7: BMI270, MicroMod_Extension:XDCR_BMI270, F.Cu at (152.0, 106.7)
- added U8: BMP384, MicroMod_Extension:PQFN45P200X200X100-10N, F.Cu at (155.8, 106.9)
- C18: footprint Capacitor_SMD:C_0402_1005Metric -> Capacitor_SMD:C_0805_2012Metric
- J1, U1: moved to B.Cu
- L2: value 2nH -> 1uH
- R11: value 510k -> 470k
- R14: value 430K -> 470k
- R15: value 82K -> 90.9k
- moved R10 70.7 mm to (139.6, 129.7), turned to 180 degrees
- moved C10 67.7 mm to (139.6, 121.6)
- moved C8 67.7 mm to (139.6, 119.6)
- moved D4 60.5 mm to (137.3, 131.4), turned to 180 degrees
- moved R1 60.5 mm to (142.7, 127.4), turned to 180 degrees
- moved C9 58.5 mm to (137.4, 119.6)
- moved J1 56.7 mm to (197.7, 96.6)
- moved SW1 53.6 mm to (162.3, 130.4)
- moved R9 53.0 mm to (139.6, 130.9), turned to 180 degrees
- moved FL1 52.6 mm to (156.1, 122.7), turned to 270 degrees
- moved U1 52.5 mm to (204.3, 87.9)
- moved FL2 52.4 mm to (162.8, 122.7), turned to 90 degrees
- moved C7 52.0 mm to (137.2, 121.4)
- moved L4 50.3 mm to (161.4, 117.1), turned to 90 degrees
- moved R2 49.5 mm to (145.1, 109.6)
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Connections:
- C1 pad 1: Net-(C1-Pad1) -> /VCCI
- C1 pad 2: Net-(C1-Pad2) -> GND
- J2 pad A6: /OTG_FS_D- -> /OTG_FS_D+
- J2 pad A7: /OTG_FS_D+ -> /OTG_FS_D-
- J2 pad B6: /OTG_FS_D- -> /OTG_FS_D+
- L2 pad 1: Net-(L2-Pad1) -> /VCCI
- L2 pad 2: Net-(L2-Pad2) -> /VCC
- U2 pad 31: Net-(FL1-Pad3) -> Net-(FL1-Pad4)
- U2 pad 32: Net-(FL1-Pad4) -> Net-(FL1-Pad3)
Other:
- copper layers 2 -> 4

Commit message: update
Parts:
- added J10: 2199230-4, MicroMod_Extension:M.2-CARD-E-22, B.Cu at (145.8, 51.8)
- added TP4: TestPoint, TestPoint:TestPoint_Plated_Hole_D3.0mm, F.Cu at (129.5, 48.3)
- added TP5: TestPoint, TestPoint:TestPoint_Plated_Hole_D3.0mm, F.Cu at (129.5, 78.7)
- added TP6: TestPoint, TestPoint:TestPoint_Plated_Hole_D3.0mm, F.Cu at (160.0, 48.3)
- added TP7: TestPoint, TestPoint:TestPoint_Plated_Hole_D3.0mm, F.Cu at (160.0, 78.7)
- added TP8: TestPoint, MicroMod_Extension:97730256330R, B.Cu at (149.9, 75.7)
- J2: moved to B.Cu
- U1: moved to F.Cu
- moved TP3 86.2 mm to (143.9, 49.0)
- moved L5 84.6 mm to (131.8, 54.7), turned to 180 degrees
- moved C19 83.8 mm to (137.8, 51.8)
- moved C22 83.8 mm to (143.9, 50.8)
- moved U5 83.8 mm to (140.8, 51.3)
- moved C18 83.5 mm to (134.5, 57.5), turned to 180 degrees
- moved TP2 83.3 mm to (142.1, 57.4)
- moved U4 81.0 mm to (131.2, 58.2), turned to 90 degrees
- moved C20 81.0 mm to (137.8, 59.8)
- moved U6 80.8 mm to (140.8, 60.6)
- moved R14 80.5 mm to (133.2, 60.5)
- moved R15 80.5 mm to (133.2, 61.7)
- moved C21 79.9 mm to (143.9, 61.2)
- moved C25 79.9 mm to (146.4, 61.2)
- moved L2 79.9 mm to (145.2, 61.2)
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
Commit message: update pcb
Parts:
- removed C10: 1u, Capacitor_SMD:C_0402_1005Metric
- removed C8: 100n, Capacitor_SMD:C_0402_1005Metric
- removed J10: 2199230-4, MicroMod_Extension:M.2-CARD-E-22
- C12, C17, C9, D5, R13, R2, R3, R6, R7: moved to B.Cu
- J4: footprint Connector_PinHeader_2.54mm:PinHeader_1x04_P2.54mm_Vertical -> Connector_JST:JST_SUR_SM04B-SURS-TF_1x04-1MP_P0.80mm_Horizontal; moved to B.Cu
- J5, J6: footprint MicroMod_Extension:JST_SUR_BM08B-SURS-TF_1x08-1MP_P0.80mm_Vertical -> Connector_JST:JST_SUR_BM08B-SURS-TF_1x08-1MP_P0.80mm_Vertical; moved to B.Cu
- J8, J9: footprint MicroMod_Extension:JST_SUR_BM04B-SURS-TF_1x04-1MP_P0.80mm_Vertical -> Connector_JST:JST_SUR_SM04B-SURS-TF_1x04-1MP_P0.80mm_Horizontal; moved to B.Cu
- TP4, TP5, TP6, TP7: value TestPoint -> Mount Hole
- TP8: value TestPoint -> Mount Hole; footprint MicroMod_Extension:97730256330R -> Mounting_Wuerth:Mounting_Wuerth_WA-SMSI-M2_H2.5mm_9774025243
- moved C9 73.3 mm to (138.2, 46.4)
- moved SW1 51.8 mm to (146.7, 81.0)
- moved C7 51.0 mm to (144.7, 71.0)
- moved J7 48.6 mm to (130.8, 52.6), turned to 90 degrees
- moved R3 46.8 mm to (137.0, 64.0), turned to 90 degrees
- moved R2 44.1 mm to (137.0, 66.2), turned to 90 degrees
- moved J5 42.0 mm to (127.4, 57.3), turned to 270 degrees
- moved C6 41.7 mm to (136.9, 78.2)
- moved D5 40.0 mm to (134.0, 77.6), turned to 90 degrees
- moved R6 39.7 mm to (136.5, 67.9)
- moved R7 39.7 mm to (138.6, 67.9)
- moved J8 38.4 mm to (161.9, 65.2), turned to 270 degrees
- moved D4 36.8 mm to (154.7, 47.4), turned to 90 degrees
- moved R10 35.2 mm to (156.6, 49.8), turned to 90 degrees
- moved J6 35.0 mm to (162.2, 56.3), turned to 90 degrees
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Connections:
- J2 pad B7: (no net) -> /OTG_FS_D-
- J8 pad 1: /VCC -> Net-(J8-Pad1)
- J9 pad 1: /VCC -> Net-(J9-Pad1)
Routing:
- net GND: track 0.00 -> 50.3 mm, vias 0 -> 23
- net /VCC: track 0.00 -> 46.5 mm, vias 0 -> 5
- net BATT: track 0.00 -> 27.7 mm, vias 0 -> 3
- net /VCCI: track 0.00 -> 23.9 mm
- net Net-(C18-Pad2): track 0.00 -> 19.7 mm
- net /VCC_NRF: track 0.00 -> 19.2 mm, vias 0 -> 5
- net /VEN_D: track 0.00 -> 12.7 mm, vias 0 -> 1
- net /SWITCH: track 0.00 -> 11.3 mm
- net /IMU_SDA: track 0.00 -> 10.5 mm, vias 0 -> 1
- net /PA_SW_ANT: track 0.00 -> 9.86 mm
- net /PA_MODE: track 0.00 -> 9.40 mm
- net /PA_RXEN: track 0.00 -> 8.77 mm
- net /IMU_SCL: track 0.00 -> 8.74 mm, vias 0 -> 2
- net Net-(FL2-Pad2): track 0.00 -> 8.74 mm
- net Net-(C3-Pad1): track 0.00 -> 8.49 mm
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Other:
- board outline added: 38.4 x 38.4 mm
- net class Default: clearance 0.2032 -> 0.1524
- rule trace_clearance: 0.2032 -> 0.1524

Commit message: update pcb
Parts:
- J7: value Conn_01x02 -> Conn_01x04; footprint Connector_PinHeader_2.54mm:PinHeader_1x02_P2.54mm_Vertical -> Connector_JST:JST_SUR_SM04B-SURS-TF_1x04-1MP_P0.80mm_Horizontal; moved to B.Cu
- R2, R3: moved to F.Cu
- moved J7 29.3 mm to (138.9, 80.8), turned to 180 degrees
- moved J4 11.0 mm to (150.0, 80.8)
- moved R3 7.82 mm to (130.4, 68.2), turned to 180 degrees
- moved R2 7.38 mm to (130.4, 69.5), turned to 180 degrees
- moved SW1 2.04 mm to (144.7, 81.2)
- moved R6 1.65 mm to (136.5, 66.3)
- moved R7 1.65 mm to (138.6, 66.3)
- moved TP1 0.28 mm to (135.0, 60.6)
- moved L5 0.13 mm to (131.8, 55.8)
Connections:
- J7 pad 1: BATT -> Net-(J7-Pad1)
- J7 pad 2: GND -> /NRF_RX2
- U2 pad 17: Net-(U2-Pad17) -> /NRF_TX2
- U2 pad 18: Net-(U2-Pad18) -> /NRF_RX2
Routing:
- net GND: track 50.3 -> 121.8 mm, vias 23 -> 71
- net VBUS: track 0.60 -> 47.0 mm, vias 0 -> 3
- net /OTG_FS_D-: track 2.52 -> 43.8 mm, vias 0 -> 2
- net /OTG_FS_D+: track 2.52 -> 42.3 mm, vias 0 -> 2
- net /NRF_RX: track 0.00 -> 31.0 mm, vias 0 -> 2
- net /NRF_CTRL: track 0.00 -> 30.6 mm, vias 0 -> 2
- net /MOTOR2: track 0.00 -> 28.9 mm, vias 0 -> 2
- net /VCC: track 46.5 -> 74.6 mm, vias 5 -> 8
- net /E_TX2: track 0.00 -> 27.8 mm
- net /NRF_TX: track 0.00 -> 27.8 mm, vias 0 -> 2
- net Net-(C18-Pad2): track 19.7 -> 47.0 mm, vias 0 -> 1
- net /E_RX2: track 0.00 -> 26.5 mm
- net /E_SDA: track 0.00 -> 24.4 mm, vias 0 -> 2
- net /MOTOR1: track 2.10 -> 26.0 mm, vias 1 -> 2
- net /PM_PGOOD: track 0.00 -> 23.1 mm, vias 0 -> 4
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- added copper zone on In1.Cu, net /VCC_NRF
- added copper zone on B.Cu, net GND
- added copper zone on F.Cu, net GND
- added copper zone on In2.Cu, net GND

Commit message: finish version 1.0
Parts:
- added J10: Conn_01x02, MicroMod_Extension:BATTARY, F.Cu at (124.7, 54.2)
- moved J3 10.7 mm to (162.1, 61.6)
- moved C11 2.03 mm to (155.8, 68.8)
- moved E1 2.03 mm to (161.5, 68.8)
- moved L1 2.03 mm to (157.9, 68.8)
- moved L3 2.03 mm to (157.4, 70.5)
Connections:
- FL2 pad 2: Net-(FL2-Pad2) -> Net-(C11-Pad2)
- FL3 pad 2: Net-(C11-Pad2) -> Net-(FL3-Pad2)
- J3 pad 1: Net-(FL2-Pad2) -> Net-(FL3-Pad2)
Routing:
- net Net-(FL3-Pad2): track 0.00 -> 11.0 mm
- net Net-(FL2-Pad2): track 8.74 -> 0.00 mm
- net GND: track 121.8 -> 118.2 mm, vias 71 -> 115
